Commit message: Pose goal works

File: src/astra_arm_urdf/urdf/astra_arm_urdf.urdf (robot description, URDF)
Before this commit: robot astra_arm_urdf, 10 links, 9 joints
Links:
- removed link ee_rotation_z
- added link robot_ee
- link ee_rotation_x: mass 0.001 -> None; geometry 
- link ee_rotation_y: mass 0.001 -> None; geometry 
Joints:
- joint ee_rotation_joint_x: limit (none) -> lower=-3.1416 upper=3.1416 effort=1 velocity=1; type continuous -> revolute
- joint ee_rotation_joint_y: limit (none) -> lower=-3.1416 upper=3.1416 effort=1 velocity=1; type continuous -> revolute
- joint ee_rotation_joint_z: child ee_rotation_z -> robot_ee; limit (none) -> lower=-3.1416 upper=3.1416 effort=1 velocity=1; type continuous -> revolute

Commit message: Revert

File: src/astra_arm_urdf/urdf/astra_arm_urdf.urdf (robot description, URDF)
Before this commit: robot astra_arm_urdf, 10 links, 9 joints
Links:
- link base_link: mass 0.21715 -> 0.21714940667968
- link ee_link: mass 0.0207769023885776 -> 0.0209019024310684
- link extra_wrist_link: mass 0.022704688254789 -> 0.0227046882547889
- link shoulder_link: mass 0.1236 -> 0.123597949087119
Joints:
- joint ee_joint: origin xyz=0.045444 0.0025 0.012135 rpy=0 0 0 -> xyz=0.11955 0.0032766 0.0078437 rpy=0 0 0

Commit message: x-rotation

File: src/astra_arm_urdf/urdf/astra_arm_urdf.urdf (robot description, URDF)
Before this commit: robot astra_arm_urdf, 10 links, 9 joints
Links:
- removed link ee_rotation_y
- removed link robot_ee
Joints:
- removed joint ee_rotation_joint_y
- removed joint ee_rotation_joint_z

File: src/xrotation/config/astra_arm_urdf.ros2_control.xacro (robot description, xacro)
@@ -43,4 +43,11 @@
                 <state_interface name="velocity"/>
             </joint>
+            <joint name="ee_rotation_joint_x">
+                <command_interface name="position"/>
+                <state_interface name="position">
+                  <param name="initial_value">${initial_positions['ee_rotation_joint_x']}</param>
+                </state_interface>
+                <state_interface name="velocity"/>
+            </joint>
         </ros2_control>
     </xacro:macro>
