Commit message: All good

File: src/arm_config/config/astra_arm_urdf.ros2_control.xacro (robot description, xacro)
@@ -13,5 +13,4 @@
                   <param name="initial_value">${initial_positions['shoulder_joint']}</param>
                 </state_interface>
-                <state_interface name="velocity"/>
             </joint>
             <joint name="upperarm_joint">
@@ -20,5 +19,4 @@
                   <param name="initial_value">${initial_positions['upperarm_joint']}</param>
                 </state_interface>
-                <state_interface name="velocity"/>
             </joint>
             <joint name="elbow_joint">
@@ -27,5 +25,4 @@
                   <param name="initial_value">${initial_positions['elbow_joint']}</param>
                 </state_interface>
-                <state_interface name="velocity"/>
             </joint>
             <joint name="wrist_joint">
@@ -34,5 +31,4 @@
                   <param name="initial_value">${initial_positions['wrist_joint']}</param>
                 </state_interface>
-                <state_interface name="velocity"/>
             </joint>
             <joint name="extra_wrist_joint">
@@ -41,5 +37,4 @@
                   <param name="initial_value">${initial_positions['extra_wrist_joint']}</param>
                 </state_interface>
-                <state_interface name="velocity"/>
             </joint>
             <joint name="ee_rotation_joint_x">
@@ -48,5 +43,4 @@
                   <param name="initial_value">${initial_positions['ee_rotation_joint_x']}</param>
                 </state_interface>
-                <state_interface name="velocity"/>
             </joint>
         </ros2_control>

File: src/astra_arm_urdf/urdf/astra_arm_urdf.urdf (robot description, URDF)
Before this commit: robot astra_arm_urdf, 8 links, 7 joints
Links:
- added link world
Joints:
- added joint world_joint: type fixed, parent world, child base_link, origin xyz=0 0 0 rpy=0 0 0
